Commit message: added gazebo control

File: colcon_ws/src/rover/description/robot.urdf.xacro (robot description, xacro)
@@ -2,3 +2,4 @@
 <robot xmlns:xacro="http://www.ros.org/wiki/xacro"  name="robot">
     <xacro:include filename="robot_core.urdf.xacro" />
+    <xacro:include filename="gazebo_control.urdf.xacro" />
 </robot>

File: colcon_ws/src/rover/description/robot_core.urdf.xacro (robot description, xacro)
@@ -38,7 +38,10 @@
         </collision>
         <xacro:inertial_box mass="5.0" x="0.450" y="0.23" z="0.18">
-            <origin xyz="0.225 0 0.09" rpy="0 0 0"/>
+            <origin xyz="0.225 0 0.09" rpy="0 0 0" />
         </xacro:inertial_box>
     </link>
+    <gazebo reference="chassis">
+        <material>Gazebo/White</material>
+    </gazebo>
     <!-- LEFT FRONT WHEEL LINK -->
     <joint name="left_front_wheel_joint" type="continuous">
@@ -47,4 +50,6 @@
         <origin xyz="0.175 0.175 .045" rpy="-${pi/2} 0 0" />
         <axis xyz="0 0 1" />
+        <limit effort="1" velocity="1" />
+        <joint_properties damping="1.0" friction="1.0" />
     </joint>
     <link name="left_front_wheel">
@@ -53,5 +58,5 @@
                 <cylinder radius="0.1" length="0.1" />
             </geometry>
-            <material name="blue" />
+            <material name="orange" />
         </visual>
         <collision>
@@ -61,7 +66,12 @@
         </collision>
         <xacro:inertial_cylinder mass="1.5" length="0.1" radius="0.1">
-            <origin xyz="0 0 0" rpy="0 0 0"/>
+            <origin xyz="0 0 0" rpy="0 0 0" />
         </xacro:inertial_cylinder>
     </link>
+    <gazebo reference="left_front_wheel">
+        <material>Gazebo/Orange</material>
+        <mu1 value="0.9" />
+        <mu2 value="0.9" />
+    </gazebo>
     <!-- LEFT BACK WHEEL LINK -->
     <joint name="left_back_wheel_joint" type="continuous">
@@ -70,4 +80,6 @@
         <origin xyz="-0.175 0.175 .045" rpy="-${pi/2} 0 0" />
         <axis xyz="0 0 1" />
+        <limit effort="1" velocity="1" />
+        <joint_properties damping="1.0" friction="1.0" />
     </joint>
     <link name="left_back_wheel">
@@ -84,7 +96,12 @@
         </collision>
         <xacro:inertial_cylinder mass="1.5" length="0.1" radius="0.1">
-            <origin xyz="0 0 0" rpy="0 0 0"/>
+            <origin xyz="0 0 0" rpy="0 0 0" />
         </xacro:inertial_cylinder>
     </link>
+    <gazebo reference="left_back_wheel">
+        <material>Gazebo/Blue</material>
+        <mu1 value="0.9" />
+        <mu2 value="0.9" />
+    </gazebo>
     <!-- RIGHT FRONT WHEEL LINK -->
     <joint name="right_front_wheel_joint" type="continuous">
@@ -92,5 +109,7 @@
         <child link="right_front_wheel" />
         <origin xyz="0.175 -0.175 .045" rpy="${pi/2} 0 0" />
-        <axis xyz="0 0 1" />
+        <axis xyz="0 0 -1" />
+        <limit effort="1" velocity="1" />
+        <joint_properties damping="1.0" friction="1.0" />
     </joint>
     <link name="right_front_wheel">
@@ -99,5 +118,5 @@
                 <cylinder radius="0.1" length="0.1" />
             </geometry>
-            <material name="blue" />
+            <material name="orange" />
         </visual>
         <collision>
@@ -107,7 +126,12 @@
         </collision>
         <xacro:inertial_cylinder mass="1.5" length="0.1" radius="0.1">
-            <origin xyz="0 0 0" rpy="0 0 0"/>
+            <origin xyz="0 0 0" rpy="0 0 0" />
         </xacro:inertial_cylinder>
     </link>
+    <gazebo reference="right_front_wheel">
+        <material>Gazebo/Orange</material>
+        <mu1 value="0.9" />
+        <mu2 value="0.9" />
+    </gazebo>
     <!-- RIGHT BACK WHEEL LINK -->
     <joint name="right_back_wheel_joint" type="continuous">
@@ -115,5 +139,7 @@
         <child link="right_back_wheel" />
         <origin xyz="-0.175 -0.175 .045" rpy="${pi/2} 0 0" />
-        <axis xyz="0 0 1" />
+        <axis xyz="0 0 -1" />
+        <limit effort="1" velocity="1" />
+        <joint_properties damping="1.0" friction="1.0" />
     </joint>
     <link name="right_back_wheel">
@@ -130,6 +156,11 @@
         </collision>
         <xacro:inertial_cylinder mass="1.5" length="0.1" radius="0.1">
-            <origin xyz="0 0 0" rpy="0 0 0"/>
+            <origin xyz="0 0 0" rpy="0 0 0" />
         </xacro:inertial_cylinder>
     </link>
+    <gazebo reference="right_back_wheel">
+        <material>Gazebo/Blue</material>
+        <mu1 value="0.9" />
+        <mu2 value="0.9" />
+    </gazebo>
 </robot>

Commit message: added gazebo lidar

File: colcon_ws/src/rover/description/robot.urdf.xacro (robot description, xacro)
@@ -3,3 +3,4 @@
     <xacro:include filename="robot_core.urdf.xacro" />
     <xacro:include filename="gazebo_control.urdf.xacro" />
+    <xacro:include filename="lidar.urdf.xacro" />
 </robot>

File: colcon_ws/src/rover/description/robot_core.urdf.xacro (robot description, xacro)
@@ -4,4 +4,7 @@
     <material name="white">
         <color rgba="1 1 1 1" />
+    </material>
+    <material name="red">
+        <color rgba="1 0 0 1" />
     </material>
     <material name="orange">
