Commit message: preparing for real robot driving

File: colcon_ws/src/rover/description/ros2_control.urdf.xacro (robot description, xacro)
@@ -1,5 +1,51 @@
 <?xml version="1.0"?>
 <robot xmlns:xacro="http://www.ros.org/wiki/xacro">
-    <ros2_control name="GazeboSystem" type="system">
+    <ros2_control name="RoverBot" type="system">
+        <hardware>
+            <plugin>diffdrive_roboclaw/DiffDriveRoboclawHardware</plugin>
+            <param name="left_front_wheel_joint">left_front_wheel_joint</param>
+            <param name="left_back_wheel_joint">left_back_wheel_joint</param>
+            <param name="right_front_wheel_joint">right_front_wheel_joint</param>
+            <param name="right_back_wheel_joint">right_back_wheel_joint</param>
+            <param name="loop_rate">30</param>
+            <param name="device">/dev/serial/by-id/usb-03eb_USB_Roboclaw_2x30A-if00</param>
+            <param name="baud_rate">115200</param>
+            <param name="timeout_ms">1000</param>
+            <param name="enc_counts_per_rev">4096</param>
+        </hardware>
+        <joint name="left_front_wheel_joint">
+            <command_interface name="velocity">
+                <param name="min">-0.1</param>
+                <param name="max">0.1</param>
+            </command_interface>
+            <state_interface name="position" />
+            <state_interface name="velocity" />
+        </joint>
+        <joint name="left_back_wheel_joint">
+            <command_interface name="velocity">
+                <param name="min">-0.1</param>
+                <param name="max">0.1</param>
+            </command_interface>
+            <state_interface name="position" />
+            <state_interface name="velocity" />
+        </joint>
+        <joint name="right_front_wheel_joint">
+            <command_interface name="velocity">
+                <param name="min">-0.1</param>
+                <param name="max">0.1</param>
+            </command_interface>
+            <state_interface name="position" />
+            <state_interface name="velocity" />
+        </joint>
+        <joint name="right_back_wheel_joint">
+            <command_interface name="velocity">
+                <param name="min">-0.1</param>
+                <param name="max">0.1</param>
+            </command_interface>
+            <state_interface name="position" />
+            <state_interface name="velocity" />
+        </joint>
+    </ros2_control>
+    <!-- <ros2_control name="GazeboSystem" type="system">
         <hardware>
             <plugin>gazebo_ros2_control/GazeboSystem</plugin>
@@ -7,6 +53,6 @@
         <joint name="left_front_wheel_joint">
             <command_interface name="velocity" >
-                <param name="min">-10</param>
-                <param name="max">10</param>
+                <param name="min">-0.1</param>
+                <param name="max">0.1</param>
             </command_interface>
             <state_interface name="velocity" />
@@ -15,6 +61,6 @@
         <joint name="left_back_wheel_joint">
             <command_interface name="velocity" >
-                <param name="min">-10</param>
-                <param name="max">10</param>
+                <param name="min">-0.1</param>
+                <param name="max">0.1</param>
             </command_interface>
             <state_interface name="velocity" />
@@ -23,6 +69,6 @@
         <joint name="right_front_wheel_joint">
             <command_interface name="velocity" >
-                <param name="min">-10</param>
-                <param name="max">10</param>
+                <param name="min">-0.1</param>
+                <param name="max">0.1</param>
             </command_interface>
             <state_interface name="velocity" />
@@ -31,11 +77,11 @@
         <joint name="right_back_wheel_joint">
             <command_interface name="velocity" >
-                <param name="min">-10</param>
-                <param name="max">10</param>
+                <param name="min">-0.1</param>
+                <param name="max">0.1</param>
             </command_interface>
             <state_interface name="velocity" />
             <state_interface name="position" />
         </joint>
-    </ros2_control>
+    </ros2_control> -->
     <gazebo>
         <plugin name="gazebo_ros2_control" filename="libgazebo_ros2_control.so">
