Commit message: gazebo update rate, sphere collisions contacts

File: colcon_ws/src/rover/description/robot_core.urdf.xacro (robot description, xacro)
@@ -65,5 +65,5 @@
         <collision>
             <geometry>
-                <cylinder radius="0.1" length="0.1" />
+                <sphere radius="0.1" />
             </geometry>
         </collision>
@@ -95,5 +95,5 @@
         <collision>
             <geometry>
-                <cylinder radius="0.1" length="0.1" />
+                <sphere radius="0.1" />
             </geometry>
         </collision>
@@ -125,5 +125,5 @@
         <collision>
             <geometry>
-                <cylinder radius="0.1" length="0.1" />
+                <sphere radius="0.1" />
             </geometry>
         </collision>
@@ -155,5 +155,5 @@
         <collision>
             <geometry>
-                <cylinder radius="0.1" length="0.1" />
+                <sphere radius="0.1" />
             </geometry>
         </collision>

Commit message: updated controller vars

File: colcon_ws/src/rover/description/robot_core.urdf.xacro (robot description, xacro)
@@ -51,5 +51,5 @@
         <parent link="base_link" />
         <child link="left_front_wheel" />
-        <origin xyz="0.175 0.175 .045" rpy="-${pi/2} 0 0" />
+        <origin xyz="0.175 0.178 .045" rpy="-${pi/2} 0 0" />
         <axis xyz="0 0 1" />
         <limit effort="1" velocity="1" />
@@ -81,5 +81,5 @@
         <parent link="base_link" />
         <child link="left_back_wheel" />
-        <origin xyz="-0.175 0.175 .045" rpy="-${pi/2} 0 0" />
+        <origin xyz="-0.175 0.178 .045" rpy="-${pi/2} 0 0" />
         <axis xyz="0 0 1" />
         <limit effort="1" velocity="1" />
@@ -111,5 +111,5 @@
         <parent link="base_link" />
         <child link="right_front_wheel" />
-        <origin xyz="0.175 -0.175 .045" rpy="${pi/2} 0 0" />
+        <origin xyz="0.175 -0.178 .045" rpy="${pi/2} 0 0" />
         <axis xyz="0 0 -1" />
         <limit effort="1" velocity="1" />
@@ -141,5 +141,5 @@
         <parent link="base_link" />
         <child link="right_back_wheel" />
-        <origin xyz="-0.175 -0.175 .045" rpy="${pi/2} 0 0" />
+        <origin xyz="-0.175 -0.178 .045" rpy="${pi/2} 0 0" />
         <axis xyz="0 0 -1" />
         <limit effort="1" velocity="1" />

File: colcon_ws/src/rover/description/ros2_control.urdf.xacro (robot description, xacro)
@@ -17,6 +17,6 @@
         <joint name="left_front_wheel_joint">
             <command_interface name="velocity">
-                <param name="min">-0.1</param>
-                <param name="max">0.1</param>
+                <param name="min">-10.0</param>
+                <param name="max">10.0</param>
             </command_interface>
             <state_interface name="position" />
@@ -25,6 +25,6 @@
         <joint name="left_back_wheel_joint">
             <command_interface name="velocity">
-                <param name="min">-0.1</param>
-                <param name="max">0.1</param>
+                <param name="min">-10.0</param>
+                <param name="max">10.0</param>
             </command_interface>
             <state_interface name="position" />
@@ -33,6 +33,6 @@
         <joint name="right_front_wheel_joint">
             <command_interface name="velocity">
-                <param name="min">-0.1</param>
-                <param name="max">0.1</param>
+                <param name="min">-10.0</param>
+                <param name="max">10.0</param>
             </command_interface>
             <state_interface name="position" />
@@ -41,6 +41,6 @@
         <joint name="right_back_wheel_joint">
             <command_interface name="velocity">
-                <param name="min">-0.1</param>
-                <param name="max">0.1</param>
+                <param name="min">-10.0</param>
+                <param name="max">10.0</param>
             </command_interface>
             <state_interface name="position" />
@@ -57,6 +57,6 @@
         <joint name="left_front_wheel_joint">
             <command_interface name="velocity" >
-                <param name="min">-0.1</param>
-                <param name="max">0.1</param>
+                <param name="min">-10.0</param>
+                <param name="max">10.0</param>
             </command_interface>
             <state_interface name="velocity" />
@@ -65,6 +65,6 @@
         <joint name="left_back_wheel_joint">
             <command_interface name="velocity" >
-                <param name="min">-0.1</param>
-                <param name="max">0.1</param>
+                <param name="min">-10.0</param>
+                <param name="max">10.0</param>
             </command_interface>
             <state_interface name="velocity" />
@@ -73,6 +73,6 @@
         <joint name="right_front_wheel_joint">
             <command_interface name="velocity" >
-                <param name="min">-0.1</param>
-                <param name="max">0.1</param>
+                <param name="min">-10.0</param>
+                <param name="max">10.0</param>
             </command_interface>
             <state_interface name="velocity" />
@@ -81,6 +81,6 @@
         <joint name="right_back_wheel_joint">
             <command_interface name="velocity" >
-                <param name="min">-0.1</param>
-                <param name="max">0.1</param>
+                <param name="min">-10.0</param>
+                <param name="max">10.0</param>
             </command_interface>
             <state_interface name="velocity" />
